File: din_isolated_SPI.kicad_pcb (KiCad board)
At the start: 2 copper layers, 31.8 x 40.5 mm, 19 parts, among them J1 CONN_01X10, U1 SI8661AB-B-IS1, U4 WeMos_mini

Commit message: PCB submitted to OSH Park.  BoM created.
Parts:
- removed LOGO1: Logo_Open_Hardware_Small, Symbols:OSHW-Symbol_6.7x6mm_SilkScreen
- removed R11, R5: 50R, Resistors_SMD:R_0603
- removed U4: WeMos_mini, wemos_d1_mini:D1_mini_board
- added MS1: ADAFRUIT_FEATHERWING_FitHome, HappyDayEnergyMonitor:ADAFRUIT_FEATHER, F.Cu at (168.9, 34.7)
- C1, C2: value 100nF -> .1u; footprint Capacitors_SMD:C_0603 -> Capacitor_SMD:C_0805_2012Metric
- G1: moved to F.Cu
- R1, R10, R12, R2, R3, R4, R6, R7, R8, R9: value 50R -> 47; footprint Resistors_SMD:R_0603 -> Resistor_SMD:R_0805_2012Metric
- moved G1 93.7 mm to (42.4, 33.7), turned to 0 degrees
- moved R3 58.4 mm to (175.9, 40.9), turned to 270 degrees
- moved R4 47.4 mm to (175.9, 35.7), turned to 270 degrees
- moved C2 47.4 mm to (175.3, 44.9)
- moved C1 47.3 mm to (175.3, 53.5), turned to 270 degrees
- moved R7 46.6 mm to (174.1, 57.3)
- moved R2 46.2 mm to (162.7, 41.5)
- moved R1 46.1 mm to (162.5, 38.3)
- moved R8 45.6 mm to (171.3, 57.3)
- moved U1 45.5 mm to (168.3, 50.1)
- moved J1 44.9 mm to (177.7, 62.9)
- moved R9 44.9 mm to (168.9, 57.3)
- moved R12 44.2 mm to (163.5, 57.3)
- moved R10 44.0 mm to (166.3, 57.3)
- moved R6 43.4 mm to (162.5, 44.7)
Connections:
- net 3V3_C renamed 3V3_CPU
- net 3V3_I renamed 3V3_M
- net CLK_E renamed SCLK_M
- net CS0_E renamed CS0_M
- net CS1_E renamed CS1_M
- net GND_C renamed GND_CPU
- net GND_I renamed GND_M
- net MISO_E renamed MISO_M
- net MOSI_E renamed MOSI_M
- J1 pad 3: CS2_E -> (no net)
- R1 pad 2: CLK_W -> CLK_C
- R2 pad 2: MOSI_W -> MOSI_C
- R3 pad 2: CS0_W -> CS0_C
- R4 pad 2: CS1_W -> CS1_C
- R6 pad 2: MISO_W -> MISO_C
- U1 pad 11: Net-(R11-Pad2) -> (no net)
- U1 pad 6: Net-(R5-Pad1) -> (no net)
Routing:
- net Net-(R4-Pad1): track 18.3 -> 37.3 mm, vias 2 -> 0
- net Net-(R5-Pad1): track 16.3 -> 0.00 mm
- net Net-(R3-Pad1): track 11.7 -> 24.6 mm, vias 2 -> 0
- net CS2_E: track 10.8 -> 0.00 mm
- net GND_CPU: track 30.4 -> 20.1 mm, vias 31 -> 4
- net Net-(R6-Pad1): track 11.0 -> 3.40 mm, vias 2 -> 0
- net CS0_W: track 6.61 -> 0.00 mm
- net CS1_C: track 0.00 -> 5.72 mm
- net 3V3_M: track 20.0 -> 25.7 mm, vias 1 -> 0
- net Net-(R1-Pad1): track 18.4 -> 12.8 mm, vias 2 -> 0
- net GND_M: track 7.44 -> 1.99 mm, vias 4 -> 2
- net MOSI_W: track 5.27 -> 0.00 mm
- net CS2_W: track 5.06 -> 0.00 mm
- net Net-(R2-Pad1): track 14.2 -> 9.27 mm, vias 2 -> 0
- net MISO_W: track 4.82 -> 0.00 mm
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- removed copper zone on F.Cu, net GND_CPU
- removed copper zone on F.Cu, net GND_M
Other:
- board size 31.8 x 40.5 mm -> 26.4 x 51.2 mm
- board text added: "FitHome CPU v. A 03/25/2019"
- board text removed: "3V3"
- board text removed: "3V3_C"
- board text removed: "3V3_I"
- board text removed: "5V"
- board text removed: "A0"
- board text removed: "CLK"
- board text removed: "CS0"
- board text removed: "CS1"
- board text removed: "CS2"
- board text removed: "D0"
- board text removed: "D1"
- board text removed: "D2"
- board text removed: "D3"
- board text removed: "D4"
- board text removed: "D5"
- board text removed: "D6"
- board text removed: "D7"
- board text removed: "D8"
- board text removed: "GND"
- board text removed: "GND_C"
- board text removed: "GND_I"
- board text removed: "MISO"
- board text removed: "MOSI"
- board text removed: "RX"
- board text removed: "TAPR"
- board text removed: "TX"
- board text removed: "Wemos Isolated SPI Basic v1.2 23/12/2017"
- board text removed: "~RST"
